File: Schematics/files/LDO_Voltage_Regilator.sch (KiCad schematic (older format))
At the start: 18 parts, among them M1 eSim_MOS_P, M2 eSim_MOS_P, M3 eSim_MOS_N, M4 eSim_MOS_N, M5 eSim_MOS_N, M6 eSim_MOS_P, M7 eSim_MOS_N, M8 eSim_MOS_P, M9 eSim_MOS_N, U1 plot_v1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

Commit message: Updated Schematics
Parts:
- removed v3: 3.55V, R1, symbol eSim_AC
- added v1: 2.55V, R1, symbol DC
Connections:
- net GND: now also v1.2 (-)
- net VIN: now also v1.1 (+)
Changed lines of the file:
@@
 	7750 3900 8900 3900
 Connection ~ 8600 3900
+Wire Wire Line
+	8000 2750 2000 2750
+Connection ~ 2150 2750
+Text GLabel 2650 3550 0    60   Input ~ 0
+VREF
+Wire Wire Line
+	2150 2750 2150 3900
+Wire Wire Line
+	2150 4800 8600 4800
 $Comp
-L eSim_AC v3
-U 1 1 6108EB30
+L DC v1
+U 1 1 6117479A
 P 2150 4350
-F 0 "v3" H 1950 4450 60  0000 C CNN
-F 1 "3.55V" H 1950 4300 60  0000 C CNN
+F 0 "v1" H 1950 4450 60  0000 C CNN
+F 1 "2.55V" H 1950 4300 60  0000 C CNN
 F 2 "R1" H 1850 4350 60  0000 C CNN
 F 3 "" H 2150 4350 60  0000 C CNN
@@
 	1    0    0    -1
 $EndComp
-Wire Wire Line
-	2000 2750 2150 2750
-Connection ~ 2150 2750
-Text GLabel 2650 3550 0    60   Input ~ 0
-VREF
-Wire Wire Line
-	2150 3900 2150 2750
-Wire Wire Line
-	2150 2750 8000 2750
-Wire Wire Line
-	2150 4800 8600 4800
 $EndSCHEMATC
